File: Active-ADC/Active-ADC.kicad_pcb (KiCad board)
At the start: 4 copper layers, 16.6 x 30.7 mm, 20 parts, among them J1 FPGA Terminal, J2 ADC Terminal, Q1 BC847, Q2 BC847, Q3 BC847

Commit message: Finalized ADC ordering
Parts:
- added R13: 3k, Resistor_SMD:R_0805_2012Metric_Pad1.20x1.40mm_HandSolder, F.Cu at (143.3, 112.0)
- C2: value 470p -> 1n
- C3: value 68p -> 150p
- Q1, Q2, Q3: value BC847 -> BFS17NTA
- R10: value 2.5k -> 2.4k
- R2: value 18k -> 10k
- R3: value 15k -> 5.1k
- R4: value 15k -> 8.2k
- R5: value 8k -> 3.3k
- R6: value 1.1k -> 523
- R7: value 2.1k -> 3.9k
- R8: value 330 -> 1.5k
- R9: value 1.5k -> 820
- moved C2 8.32 mm to (141.5, 120.1), turned to 0 degrees
Connections:
- Q1 pad 1: /SIGMA-CHERRY -> Net-(Q1-Pad1)
Routing:
- net GND: track 60.6 -> 51.9 mm
- net Net-(C2-Pad1): track 6.78 -> 12.5 mm
- net Net-(Q1-Pad1): track 0.00 -> 3.64 mm
- net /SIGMA-CHERRY: track 8.53 -> 5.92 mm
