File: Active-ADC/Active-ADC.kicad_sch (KiCad schematic)
At the start: 18 parts, among them J1 FPGA Terminal, J2 ADC Terminal, Q1 BC847, Q2 BC847, Q3 BC847

Commit message: Added part numbers and switched footprints to SMD
Parts:
- R1, R10, R2, R3, R4, R5, R6, R7, R8, R9: footprint Resistor_THT:R_Axial_DIN0207_L6.3mm_D2.5mm_P10.16mm_Horizontal -> Resistor_SMD:R_0201_0603Metric
Changed lines of the file:
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@@
     (property "Reference" "R5" (id 0) (at 73.66 19.05 90))
     (property "Value" "56k" (id 1) (at 73.66 21.59 90))
-    (property "Footprint" "Resistor_THT:R_Axial_DIN0207_L6.3mm_D2.5mm_P10.16mm_Horizontal" (id 2) (at 73.66 27.178 90)
-      (effects (font (size 1.27 1.27)) hide)
-    )
-    (property "Datasheet" "~" (id 3) (at 73.66 25.4 0)
+    (property "Footprint" "Resistor_SMD:R_0201_0603Metric" (id 2) (at 73.66 27.178 90)
+      (effects (font (size 1.27 1.27)) hide)
+    )
+    (property "Datasheet" "P123347TR-ND" (id 3) (at 73.66 25.4 0)
       (effects (font (size 1.27 1.27)) hide)
     )
@@
       (effects (font (size 1.27 1.27)) (justify left))
     )
-    (property "Footprint" "Resistor_THT:R_Axial_DIN0207_L6.3mm_D2.5mm_P10.16mm_Horizontal" (id 2) (at 68.072 92.71 90)
+    (property "Footprint" "Resistor_SMD:R_0201_0603Metric" (id 2) (at 68.072 92.71 90)
       (effects (font (size 1.27 1.27)) hide)
     )
@@
       (effects (font (size 1.27 1.27)) (justify left))
     )
-    (property "Footprint" "Resistor_THT:R_Axial_DIN0207_L6.3mm_D2.5mm_P10.16mm_Horizontal" (id 2) (at 68.072 80.01 90)
+    (property "Footprint" "Resistor_SMD:R_0201_0603Metric" (id 2) (at 68.072 80.01 90)
       (effects (font (size 1.27 1.27)) hide)
     )
@@
     (property "Reference" "R4" (id 0) (at 60.96 19.05 90))
     (property "Value" "18k" (id 1) (at 60.96 21.59 90))
-    (property "Footprint" "Resistor_THT:R_Axial_DIN0207_L6.3mm_D2.5mm_P10.16mm_Horizontal" (id 2) (at 60.96 27.178 90)
-      (effects (font (size 1.27 1.27)) hide)
-    )
-    (property "Datasheet" "~" (id 3) (at 60.96 25.4 0)
+    (property "Footprint" "Resistor_SMD:R_0201_0603Metric" (id 2) (at 60.96 27.178 90)
+      (effects (font (size 1.27 1.27)) hide)
+    )
+    (property "Datasheet" "311-18.0KMTR-ND" (id 3) (at 60.96 25.4 0)
       (effects (font (size 1.27 1.27)) hide)
     )
@@
       (effects (font (size 1.27 1.27)) (justify left))
     )
-    (property "Footprint" "Resistor_THT:R_Axial_DIN0207_L6.3mm_D2.5mm_P10.16mm_Horizontal" (id 2) (at 50.292 125.73 90)
+    (property "Footprint" "Resistor_SMD:R_0201_0603Metric" (id 2) (at 50.292 125.73 90)
       (effects (font (size 1.27 1.27)) hide)
     )
@@
       (effects (font (size 1.27 1.27)) (justify right))
     )
-    (property "Footprint" "Resistor_THT:R_Axial_DIN0207_L6.3mm_D2.5mm_P10.16mm_Horizontal" (id 2) (at 81.788 43.18 90)
-      (effects (font (size 1.27 1.27)) hide)
-    )
-    (property "Datasheet" "~" (id 3) (at 80.01 43.18 0)
+    (property "Footprint" "Resistor_SMD:R_0201_0603Metric" (id 2) (at 81.788 43.18 90)
+      (effects (font (size 1.27 1.27)) hide)
+    )
+    (property "Datasheet" "YAG2379TR-ND" (id 3) (at 80.01 43.18 0)
       (effects (font (size 1.27 1.27)) hide)
     )
@@
       (effects (font (size 1.27 1.27)) (justify right))
     )
-    (property "Footprint" "Resistor_THT:R_Axial_DIN0207_L6.3mm_D2.5mm_P10.16mm_Horizontal" (id 2) (at 56.388 31.75 90)
-      (effects (font (size 1.27 1.27)) hide)
-    )
-    (property "Datasheet" "~" (id 3) (at 54.61 31.75 0)
+    (property "Footprint" "Resistor_SMD:R_0201_0603Metric" (id 2) (at 56.388 31.75 90)
+      (effects (font (size 1.27 1.27)) hide)
+    )
+    (property "Datasheet" "311-18.0KMTR-ND" (id 3) (at 54.61 31.75 0)
       (effects (font (size 1.27 1.27)) hide)
     )
@@
     (property "Reference" "R2" (id 0) (at 48.26 19.05 90))
     (property "Value" "36k" (id 1) (at 48.26 21.59 90))
-    (property "Footprint" "Resistor_THT:R_Axial_DIN0207_L6.3mm_D2.5mm_P10.16mm_Horizontal" (id 2) (at 48.26 27.178 90)
-      (effects (font (size 1.27 1.27)) hide)
-    )
-    (property "Datasheet" "~" (id 3) (at 48.26 25.4 0)
+    (property "Footprint" "Resistor_SMD:R_0201_0603Metric" (id 2) (at 48.26 27.178 90)
+      (effects (font (size 1.27 1.27)) hide)
+    )
+    (property "Datasheet" "YAG2626TR-ND" (id 3) (at 48.26 25.4 0)
       (effects (font (size 1.27 1.27)) hide)
     )
@@
     (property "Reference" "R1" (id 0) (at 35.56 19.05 90))
     (property "Value" "100" (id 1) (at 35.56 21.59 90))
-    (property "Footprint" "Resistor_THT:R_Axial_DIN0207_L6.3mm_D2.5mm_P10.16mm_Horizontal" (id 2) (at 35.56 27.178 90)
-      (effects (font (size 1.27 1.27)) hide)
-    )
-    (property "Datasheet" "~" (id 3) (at 35.56 25.4 0)
+    (property "Footprint" "Resistor_SMD:R_0201_0603Metric" (id 2) (at 35.56 27.178 90)
+      (effects (font (size 1.27 1.27)) hide)
+    )
+    (property "Datasheet" "311-100MTR-ND" (id 3) (at 35.56 25.4 0)
       (effects (font (size 1.27 1.27)) hide)
     )
@@
       (effects (font (size 1.27 1.27)) (justify left))
     )
-    (property "Footprint" "Resistor_THT:R_Axial_DIN0207_L6.3mm_D2.5mm_P10.16mm_Horizontal" (id 2) (at 50.292 97.79 90)
+    (property "Footprint" "Resistor_SMD:R_0201_0603Metric" (id 2) (at 50.292 97.79 90)
       (effects (font (size 1.27 1.27)) hide)
     )
@@
     )
     (path "/da851561-7fdb-4f61-b0c2-2413cfd57a0f"
-      (reference "R1") (unit 1) (value "100") (footprint "Resistor_THT:R_Axial_DIN0207_L6.3mm_D2.5mm_P10.16mm_Horizontal")
+      (reference "R1") (unit 1) (value "100") (footprint "Resistor_SMD:R_0201_0603Metric")
     )
     (path "/a4a8430c-d7a1-47ce-bbb3-0b02aed0c1eb"
-      (reference "R2") (unit 1) (value "36k") (footprint "Resistor_THT:R_Axial_DIN0207_L6.3mm_D2.5mm_P10.16mm_Horizontal")
+      (reference "R2") (unit 1) (value "36k") (footprint "Resistor_SMD:R_0201_0603Metric")
     )
     (path "/88afc6d6-80c2-449c-adb0-b4bcf7eec011"
-      (reference "R3") (unit 1) (value "18k") (footprint "Resistor_THT:R_Axial_DIN0207_L6.3mm_D2.5mm_P10.16mm_Horizontal")
+      (reference "R3") (unit 1) (value "18k") (footprint "Resistor_SMD:R_0201_0603Metric")
     )
     (path "/699138f6-237a-4b8a-a4d4-7fb9091d901b"
-      (reference "R4") (unit 1) (value "18k") (footprint "Resistor_THT:R_Axial_DIN0207_L6.3mm_D2.5mm_P10.16mm_Horizontal")
+      (reference "R4") (unit 1) (value "18k") (footprint "Resistor_SMD:R_0201_0603Metric")
     )
     (path "/0456c7de-9f79-46f5-a17e-4fa13a1b0cfc"
-      (reference "R5") (unit 1) (value "56k") (footprint "Resistor_THT:R_Axial_DIN0207_L6.3mm_D2.5mm_P10.16mm_Horizontal")
+      (reference "R5") (unit 1) (value "56k") (footprint "Resistor_SMD:R_0201_0603Metric")
     )
     (path "/84aecc63-06ed-478f-8f5f-d0d1edf5fbec"
-      (reference "R6") (unit 1) (value "110") (footprint "Resistor_THT:R_Axial_DIN0207_L6.3mm_D2.5mm_P10.16mm_Horizontal")
+      (reference "R6") (unit 1) (value "110") (footprint "Resistor_SMD:R_0201_0603Metric")
     )
     (path "/f2a977c8-30ef-4319-82c2-32f34a4a3175"
-      (reference "R7") (unit 1) (value "2.1k") (footprint "Resistor_THT:R_Axial_DIN0207_L6.3mm_D2.5mm_P10.16mm_Horizontal")
+      (reference "R7") (unit 1) (value "2.1k") (footprint "Resistor_SMD:R_0201_0603Metric")
     )
     (path "/745cd236-ebd5-45a2-9f15-f3ef3d7dae9c"
-      (reference "R8") (unit 1) (value "375") (footprint "Resistor_THT:R_Axial_DIN0207_L6.3mm_D2.5mm_P10.16mm_Horizontal")
+      (reference "R8") (unit 1) (value "375") (footprint "Resistor_SMD:R_0201_0603Metric")
     )
     (path "/38d17884-57d2-4dc7-9a53-9bb47fd2d837"
-      (reference "R9") (unit 1) (value "1.5k") (footprint "Resistor_THT:R_Axial_DIN0207_L6.3mm_D2.5mm_P10.16mm_Horizontal")
+      (reference "R9") (unit 1) (value "1.5k") (footprint "Resistor_SMD:R_0201_0603Metric")
     )
     (path "/2b56ea83-9e8a-4d22-a128-e140e248933c"
-      (reference "R10") (unit 1) (value "2.5k") (footprint "Resistor_THT:R_Axial_DIN0207_L6.3mm_D2.5mm_P10.16mm_Horizontal")
-    )
-  )
+      (reference "R10") (unit 1) (value "2.5k") (footprint "Resistor_SMD:R_0201_0603Metric")
+    )
+  )

Commit message: Updated part numbers
Parts:
- C1, C2: footprint Capacitor_THT:CP_Radial_D7.5mm_P2.50mm -> Capacitor_SMD:C_0201_0603Metric
- C3: footprint Capacitor_THT:CP_Radial_D7.5mm_P2.50mm -> Capacitor_SMD:C_0402_1005Metric
Changed lines of the file:
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@@
       (effects (font (size 1.27 1.27)) (justify left))
     )
-    (property "Footprint" "Capacitor_THT:CP_Radial_D7.5mm_P2.50mm" (id 2) (at 42.8752 35.56 0)
-      (effects (font (size 1.27 1.27)) hide)
-    )
-    (property "Datasheet" "~" (id 3) (at 41.91 31.75 0)
+    (property "Footprint" "Capacitor_SMD:C_0201_0603Metric" (id 2) (at 42.8752 35.56 0)
+      (effects (font (size 1.27 1.27)) hide)
+    )
+    (property "Datasheet" "478-5266-2-ND" (id 3) (at 41.91 31.75 0)
       (effects (font (size 1.27 1.27)) hide)
     )
@@
       (effects (font (size 1.27 1.27) italic) (justify left) hide)
     )
-    (property "Datasheet" "http://www.infineon.com/dgdl/Infineon-BC847SERIES_BC848SERIES_BC849SERIES_BC850SERIES-DS-v01_01-en.pdf?fileId=db3a304314dca389011541d4630a1657" (id 3) (at 54.61 86.36 0)
+    (property "Datasheet" "BFS17NTATR-ND" (id 3) (at 54.61 86.36 0)
       (effects (font (size 1.27 1.27)) (justify left) hide)
     )
@@
       (effects (font (size 1.27 1.27)) (justify left))
     )
-    (property "Footprint" "Capacitor_THT:CP_Radial_D7.5mm_P2.50mm" (id 2) (at 68.2752 35.56 0)
-      (effects (font (size 1.27 1.27)) hide)
-    )
-    (property "Datasheet" "~" (id 3) (at 67.31 31.75 0)
+    (property "Footprint" "Capacitor_SMD:C_0201_0603Metric" (id 2) (at 68.2752 35.56 0)
+      (effects (font (size 1.27 1.27)) hide)
+    )
+    (property "Datasheet" "445-12113-2-ND" (id 3) (at 67.31 31.75 0)
       (effects (font (size 1.27 1.27)) hide)
     )
@@
       (effects (font (size 1.27 1.27)) (justify left))
     )
-    (property "Footprint" "Capacitor_THT:CP_Radial_D7.5mm_P2.50mm" (id 2) (at 80.9752 35.56 0)
-      (effects (font (size 1.27 1.27)) hide)
-    )
-    (property "Datasheet" "~" (id 3) (at 80.01 31.75 0)
+    (property "Footprint" "Capacitor_SMD:C_0402_1005Metric" (id 2) (at 80.9752 35.56 0)
+      (effects (font (size 1.27 1.27)) hide)
+    )
+    (property "Datasheet" "478-1080-2-ND" (id 3) (at 80.01 31.75 0)
       (effects (font (size 1.27 1.27)) hide)
     )
@@
       (effects (font (size 1.27 1.27) italic) (justify left) hide)
     )
-    (property "Datasheet" "http://www.infineon.com/dgdl/Infineon-BC847SERIES_BC848SERIES_BC849SERIES_BC850SERIES-DS-v01_01-en.pdf?fileId=db3a304314dca389011541d4630a1657" (id 3) (at 49.53 113.03 0)
+    (property "Datasheet" "BFS17NTATR-ND" (id 3) (at 49.53 113.03 0)
       (effects (font (size 1.27 1.27)) (justify left) hide)
     )
@@
       (effects (font (size 1.27 1.27) italic) (justify left) hide)
     )
-    (property "Datasheet" "http://www.infineon.com/dgdl/Infineon-BC847SERIES_BC848SERIES_BC849SERIES_BC850SERIES-DS-v01_01-en.pdf?fileId=db3a304314dca389011541d4630a1657" (id 3) (at 67.31 105.41 0)
+    (property "Datasheet" "BFS17NTATR-ND" (id 3) (at 67.31 105.41 0)
       (effects (font (size 1.27 1.27)) (justify left) hide)
     )
@@
     )
     (path "/1e9f2ce0-6d08-46ba-8d06-09c985b358e9"
-      (reference "C1") (unit 1) (value ".1u") (footprint "Capacitor_THT:CP_Radial_D7.5mm_P2.50mm")
+      (reference "C1") (unit 1) (value ".1u") (footprint "Capacitor_SMD:C_0201_0603Metric")
     )
     (path "/c440b35e-3f7e-431c-90ab-fb12d5c34ace"
-      (reference "C2") (unit 1) (value "470p") (footprint "Capacitor_THT:CP_Radial_D7.5mm_P2.50mm")
+      (reference "C2") (unit 1) (value "470p") (footprint "Capacitor_SMD:C_0201_0603Metric")
     )
     (path "/dd02a207-fa49-45c1-8a6d-f9dc54a91fee"
-      (reference "C3") (unit 1) (value "68p") (footprint "Capacitor_THT:CP_Radial_D7.5mm_P2.50mm")
+      (reference "C3") (unit 1) (value "68p") (footprint "Capacitor_SMD:C_0402_1005Metric")
     )
     (path "/fbc3ac75-825f-438a-85e7-381ae2adaad7"
