File: Active-ADC/Active-ADC.kicad_sch (KiCad schematic)
At the start: 20 parts, among them J1 FPGA Terminal, J2 ADC Terminal, Q1 BFS17NTA, Q2 BFS17NTA, Q3 BFS17NTA

Commit message: Finalized ADC ordering
Parts:
- added R13: 3k, Resistor_SMD:R_0805_2012Metric_Pad1.20x1.40mm_HandSolder, symbol Device:R
Connections:
- net SIGMA-CHERRY: now also R13.1; no longer Q1.1 (B)
- new net: Q1.1 (B), R13.2
Changed lines of the file:
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@@
+    (stroke (width 0) (type default) (color 0 0 0 0))
+  )
+  (wire (pts (xy 29.21 113.03) (xy 33.02 113.03))
     (stroke (width 0) (type default) (color 0 0 0 0))
   )
@@
     (stroke (width 0) (type default) (color 0 0 0 0))
   )
+  (wire (pts (xy 40.64 113.03) (xy 44.45 113.03))
+    (stroke (width 0) (type default) (color 0 0 0 0))
+  )
   (wire (pts (xy 41.91 25.4) (xy 41.91 27.94))
     (stroke (width 0) (type default) (color 0 0 0 0))
@@
   )
   (polyline (pts (xy 109.22 12.7) (xy 109.22 59.69))
-    (stroke (width 0) (type default) (color 0 0 0 0))
-  )
-  (wire (pts (xy 39.37 113.03) (xy 44.45 113.03))
     (stroke (width 0) (type default) (color 0 0 0 0))
   )
@@
     (effects (font (size 1.27 1.27)) (justify right bottom))
   )
-  (label "SIGMA-CHERRY" (at 39.37 113.03 180)
+  (label "SIGMA-CHERRY" (at 29.21 113.03 180)
     (effects (font (size 1.27 1.27)) (justify right bottom))
   )
@@
       (effects (font (size 1.27 1.27)) hide)
     )
-    (property "Datasheet" "1276-2568-2-ND" (id 3) (at 41.91 31.75 0)
+    (property "Datasheet" "1276-1003-2-ND" (id 3) (at 41.91 31.75 0)
       (effects (font (size 1.27 1.27)) hide)
     )
@@
     )
     (pin "1")
+  )
+  (symbol (lib_id "Device:R") (at 36.83 113.03 90) (unit 1)
+    (in_bom yes) (on_board yes) (fields_autoplaced)
+    (property "Reference" "R13" (id 0) (at 36.83 106.68 90))
+    (property "Value" "3k" (id 1) (at 36.83 109.22 90))
+    (property "Footprint" "Resistor_SMD:R_0805_2012Metric_Pad1.20x1.40mm_HandSolder" (id 2) (at 36.83 114.808 90)
+      (effects (font (size 1.27 1.27)) hide)
+    )
+    (property "Datasheet" "311-1.50KCRTR-ND" (id 3) (at 36.83 113.03 0)
+      (effects (font (size 1.27 1.27)) hide)
+    )
+    (pin "1")
+    (pin "2")
   )
   (symbol (lib_id "Device:R") (at 265.43 25.4 0) (unit 1)
@@
       (reference "R12") (unit 1) (value "3.3k") (footprint "Resistor_SMD:R_0805_2012Metric_Pad1.20x1.40mm_HandSolder")
     )
-  )
+    (path "/e2271da3-4134-4d35-af74-1bf6dca24b06"
+      (reference "R13") (unit 1) (value "3k") (footprint "Resistor_SMD:R_0805_2012Metric_Pad1.20x1.40mm_HandSolder")
+    )
+  )
